File: simple_circuit.kicad_sch (KiCad schematic)
At the start: 1 part

Commit message: ✅ Fix reference designator display - components now show R1 instead of R?
- Fixed UUID mismatch between schematic UUID and component instances path
- Updated component instances to use schematic UUID for proper annotation
- Fixed property name casing in library cache (Description/Datasheet)
- Added logging for UUID tracking and property debugging
- Simplified test script with all required component properties

🤖 Generated with [Claude Code](https://claude.ai/code)

Co-Authored-By: Claude <noreply@anthropic.com>
Parts:
- R1: footprint (none) -> Resistor_SMD:R_0603_1608Metric; description (none) -> Resistor
Changed lines of the file:
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@@
+			)
+		)
+		(property "Footprint" "Resistor_SMD:R_0603_1608Metric"
+			(at 102.54 103.81 0)
+			(effects
+				(font
+					(size 1.27 1.27)
+				)
+				(justify left)
+				(hide yes)
+			)
+		)
+		(property "datasheet" "~"
+			(at 102.54 105.08 0)
+			(effects
+				(font
+					(size 1.27 1.27)
+				)
+				(justify left)
+				(hide yes)
+			)
+		)
+		(property "description" "Resistor"
+			(at 102.54 105.08 0)
+			(effects
+				(font
+					(size 1.27 1.27)
+				)
+				(justify left)
+				(hide yes)
 			)
 		)
@@
 		(instances
 			(project "simple_circuit"
-				(path "/b820464d-ba53-4df6-8301-e55492dc6243"
+				(path "/9bae8aa0-2a10-402d-bcd1-f83ce99fad42"
 					(reference "R1")
 					(unit 1)
