File: examples/KEEP/voltage_divider.kicad_sch (KiCad schematic)
At the start: 2 parts

Commit message: Demonstrate auto_route_pins API in voltage divider example
Updated example to show pin-to-pin auto-routing between resistors.

Before (all manual wiring):
  sch.add_wire(start=p(0, 8), end=p(0, 11))   # R1 bottom to junction
  sch.add_wire(start=p(0, 11), end=p(0, 12))  # Junction to R2 top

After (auto-route between pins):
  sch.auto_route_pins('R1', '2', 'R2', '1', routing_strategy='direct')

This demonstrates the convenient pin-to-pin connection API which:
- Automatically calculates pin positions
- Creates properly routed wires
- Handles component rotations automatically

The example now shows both manual wiring (for power connections)
and auto-routing (for component-to-component connections).

🤖 Generated with [Claude Code](https://claude.com/claude-code)

Co-Authored-By: Claude <noreply@anthropic.com>
Changed lines of the file:
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@@
 		(instances
 			(project "Example_VoltageDiv"
-				(path "/371c2d0d-60df-4e73-b9ce-fe4473bf1ba8"
+				(path "/f131e43e-874c-4758-a339-d7da6f0cb3ae"
 					(reference "#PWR01")
 					(unit 1)
@@
 		(instances
 			(project "Example_VoltageDiv"
-				(path "/371c2d0d-60df-4e73-b9ce-fe4473bf1ba8"
+				(path "/f131e43e-874c-4758-a339-d7da6f0cb3ae"
 					(reference "#PWR02")
 					(unit 1)
@@
 		(instances
 			(project "Example_VoltageDiv"
-				(path "/371c2d0d-60df-4e73-b9ce-fe4473bf1ba8"
+				(path "/f131e43e-874c-4758-a339-d7da6f0cb3ae"
 					(reference "R1")
 					(unit 1)
@@
 		(instances
 			(project "Example_VoltageDiv"
-				(path "/371c2d0d-60df-4e73-b9ce-fe4473bf1ba8"
+				(path "/f131e43e-874c-4758-a339-d7da6f0cb3ae"
 					(reference "R2")
 					(unit 1)
@@
 	(wire
 		(pts
-			(xy 25.4 35.56) (xy 25.4 39.37)
+			(xy 25.4 48.26) (xy 25.4 52.07)
 		)
 		(stroke
@@
 	(wire
 		(pts
-			(xy 25.4 39.37) (xy 25.4 40.64)
+			(xy 25.4 35.56) (xy 25.4 40.64)
 		)
 		(stroke
-			(width 0)
-			(type default)
-		)
-	)
-	(wire
-		(pts
-			(xy 25.4 48.26) (xy 25.4 52.07)
-		)
-		(stroke
